File: jamma_mahjong/jamma_mahjong.sch (KiCad schematic (older format))
At the start: 3 parts, among them J1 Jamma_Connector, J2 Mahjong_Connector, J3 Conn_02x07_Odd_Even

Commit message: x
Parts:
- added JMP1: SolderJumper_2_Open, Resistor_SMD:R_0805_2012Metric_Pad1.20x1.40mm_HandSolder, symbol Jumper:SolderJumper_2_Open
- added SW1: SW_SPDT, SPDT:A101SYCQ04, symbol Switch:SW_SPDT
Connections:
- net -5V: now also JMP1.2 (B); no longer J1.E (Pin_E)
- net GND: now also J1.14 (Pin_14), SW1.3 (C)
- net -5V_M: now reaches J2.24 (Pin_24)
- net -5V_M: now also JMP1.1 (A)
- net SPK- renamed JAMMA_SPK-
- net JAMMA_SPK-: now also SW1.2 (B); no longer J2.10 (Pin_10)
- new net JONG_SPK-: J2.10 (Pin_10), SW1.1 (A)
- no-connect marks 34 -> 33
Changed lines of the file:
@@
 Text GLabel 2150 2000 0    50   Input ~ 0
--5V
-Text GLabel 2650 2000 2    50   Input ~ 0
 -5V
 Text GLabel 2150 2100 0    50   Input ~ 0
@@
 SPK+
 Text GLabel 2650 2500 2    50   Input ~ 0
-SPK-
+JAMMA_SPK-
 Text GLabel 4400 2500 0    50   Input ~ 0
-SPK-
+JONG_SPK-
 Text GLabel 4400 2200 0    50   Input ~ 0
 TEST
@@
 NoConn ~ 4900 3300
 NoConn ~ 4400 3300
-NoConn ~ 4400 3900
-NoConn ~ 4900 3900
 Text GLabel 4900 2100 2    50   Input ~ 0
 SERVICE
@@
 Text GLabel 2150 3000 0    50   Input ~ 0
 TEST
-NoConn ~ 2150 2900
 NoConn ~ 2650 3000
 $Comp
@@
 Text GLabel 2150 3700 0    50   Input ~ 0
 COM4-7
+Wire Wire Line
+	2150 2900 1750 2900
+Wire Wire Line
+	1750 2900 1750 2950
+$Comp
+L power:GND #PWR0110
+U 1 1 61CCDF98
+P 1750 2950
+F 0 "#PWR0110" H 1750 2700 50  0001 C CNN
+F 1 "GND" H 1755 2777 50  0000 C CNN
+F 2 "" H 1750 2950 50  0001 C CNN
+F 3 "" H 1750 2950 50  0001 C CNN
+	1    1750 2950
+	1    0    0    -1
+$EndComp
+$Comp
+L Jumper:SolderJumper_2_Open JMP1
+U 1 1 61CD2BFC
+P 7850 2700
+F 0 "JMP1" H 7850 2905 50  0000 C CNN
+F 1 "SolderJumper_2_Open" H 7850 2814 50  0000 C CNN
+F 2 "Resistor_SMD:R_0805_2012Metric_Pad1.20x1.40mm_HandSolder" H 7850 2700 50  0001 C CNN
+F 3 "~" H 7850 2700 50  0001 C CNN
+	1    7850 2700
+	1    0    0    -1
+$EndComp
+Text GLabel 4400 3900 0    50   Input ~ 0
+-5V_M
+NoConn ~ 4900 3900
+NoConn ~ 2650 2000
+Text GLabel 7700 2700 0    50   Input ~ 0
+-5V_M
+Text GLabel 8000 2700 2    50   Input ~ 0
+-5V
+$Comp
+L Switch:SW_SPDT SW1
+U 1 1 61D02BFB
+P 7850 3200
+F 0 "SW1" H 7850 3485 50  0000 C CNN
+F 1 "SW_SPDT" H 7850 3394 50  0000 C CNN
+F 2 "SPDT:A101SYCQ04" H 7850 3200 50  0001 C CNN
+F 3 "~" H 7850 3200 50  0001 C CNN
+	1    7850 3200
+	1    0    0    -1
+$EndComp
+Text GLabel 7650 3200 0    50   Input ~ 0
+JAMMA_SPK-
+Text GLabel 8050 3100 2    50   Input ~ 0
+JONG_SPK-
+$Comp
+L power:GND #PWR0111
+U 1 1 61D06E40
+P 8150 3400
+F 0 "#PWR0111" H 8150 3150 50  0001 C CNN
+F 1 "GND" H 8155 3227 50  0000 C CNN
+F 2 "" H 8150 3400 50  0001 C CNN
+F 3 "" H 8150 3400 50  0001 C CNN
+	1    8150 3400
+	1    0    0    -1
+$EndComp
+Wire Wire Line
+	8050 3300 8150 3300
+Wire Wire Line
+	8150 3300 8150 3400
 $EndSCHEMATC

Commit message: x
Parts:
- added JMP2, JMP3: SolderJumper_2_Open, Resistor_SMD:R_0805_2012Metric_Pad1.20x1.40mm_HandSolder, symbol Jumper:SolderJumper_2_Open
Connections:
- net -5V: now also J1.E (Pin_E); no longer J1.5 (Pin_5)
- net -5V_M: now also J2.b (Pin_b); no longer J2.24 (Pin_24)
- net GND: now also JMP3.2 (B)
- net JAMMA_SPK-: now also JMP2.1 (A), JMP3.1 (A)
- net JONG_SPK-: now also JMP2.2 (B)
Other:
- moved on the sheet: J1, J3, JMP1, SW1

Commit message: v2
Parts:
- removed J3: Conn_02x07_Odd_Even, Connector_JST:JST_PHD_B14B-PHDSS_2x07_P2.00mm_Vertical, symbol Connector_Generic:Conn_02x07_Odd_Even
- added J3, J4: Conn_01x06, Connector_JST:JST_EH_B6B-EH-A_1x06_P2.50mm_Vertical, symbol Connector_Generic:Conn_01x06
- added J5: Conn_01x02, Connector_JST:JST_EH_B2B-EH-A_1x02_P2.50mm_Vertical, symbol Connector_Generic:Conn_01x02
Connections:
- net 5V: now also J5.1 (Pin_1)
- net COIN: now also J3.6 (Pin_6)
- net COM0-3: now also J1.U (Pin_U), J3.1 (Pin_1); no longer J1.18 (Pin_18)
- net COM1-2: now also J1.V (Pin_V), J3.2 (Pin_2); no longer J1.19 (Pin_19)
- net COM2-6: now also J1.W (Pin_W), J3.3 (Pin_3); no longer J1.20 (Pin_20)
- net COM3-10: now also J1.X (Pin_X), J3.4 (Pin_4); no longer J1.21 (Pin_21)
- net COM4-7: now also J1.Y (Pin_Y), J3.5 (Pin_5); no longer J1.22 (Pin_22)
- net GND: now also J5.2 (Pin_2)
- net KEY0-4: now also J1.17 (Pin_17), J4.1 (Pin_1); no longer J1.V (Pin_V)
- net KEY1-5: now also J1.18 (Pin_18), J4.2 (Pin_2); no longer J1.W (Pin_W)
- net KEY2-8: now also J1.19 (Pin_19), J4.3 (Pin_3); no longer J1.X (Pin_X)
- net KEY3-9: now also J1.20 (Pin_20), J4.4 (Pin_4); no longer J1.Y (Pin_Y)
- net KEY4-11: now also J1.21 (Pin_21), J4.5 (Pin_5); no longer J1.Z (Pin_Z)
- net KEY5-1: now also J1.22 (Pin_22), J4.6 (Pin_6); no longer J1.a (Pin_a)
Changed lines of the file:
@@
 NoConn ~ 2650 4100
 NoConn ~ 3150 4100
-NoConn ~ 2650 3200
-NoConn ~ 3150 3200
+NoConn ~ 3150 3800
+NoConn ~ 3150 3700
 NoConn ~ 3150 3900
 NoConn ~ 3150 4000
@@
 Text GLabel 4900 3800 2    50   Input ~ 0
 12V
-Text GLabel 6600 1650 2    50   Input ~ 0
-KEY0-4
-Text GLabel 6600 1750 2    50   Input ~ 0
-KEY1-5
-Text GLabel 6600 1850 2    50   Input ~ 0
-KEY2-8
-Text GLabel 6600 1950 2    50   Input ~ 0
-KEY3-9
-Text GLabel 6600 2050 2    50   Input ~ 0
-KEY4-11
-Text GLabel 6600 2150 2    50   Input ~ 0
-KEY5-1
-Text GLabel 6100 2150 0    50   Input ~ 0
-COM4-7
-Text GLabel 6100 2050 0    50   Input ~ 0
-COM3-10
-Text GLabel 6100 1950 0    50   Input ~ 0
-COM2-6
-Text GLabel 6100 1850 0    50   Input ~ 0
-COM1-2
-Text GLabel 6100 1750 0    50   Input ~ 0
-COM0-3
-Text GLabel 6100 1650 0    50   Input ~ 0
-COIN
-$Comp
-L power:GND #PWR0109
-U 1 1 61C03E3B
-P 7050 1550
-F 0 "#PWR0109" H 7050 1300 50  0001 C CNN
-F 1 "GND" H 7055 1377 50  0000 C CNN
-F 2 "" H 7050 1550 50  0001 C CNN
-F 3 "" H 7050 1550 50  0001 C CNN
-	1    7050 1550
-	1    0    0    -1
-$EndComp
-Wire Wire Line
-	6600 1550 7050 1550
-Text GLabel 6100 1550 0    50   Input ~ 0
-5V
-$Comp
-L Connector_Generic:Conn_02x07_Odd_Even J3
-U 1 1 61C0E561
-P 6300 1850
-F 0 "J3" H 6350 2367 50  0000 C CNN
-F 1 "Conn_02x07_Odd_Even" H 6350 2276 50  0000 C CNN
-F 2 "Connector_JST:JST_PHD_B14B-PHDSS_2x07_P2.00mm_Vertical" H 6300 1850 50  0001 C CNN
-F 3 "~" H 6300 1850 50  0001 C CNN
-	1    6300 1850
-	1    0    0    -1
-$EndComp
-Text GLabel 3150 3300 2    50   Input ~ 0
-KEY0-4
-Text GLabel 3150 3400 2    50   Input ~ 0
-KEY1-5
-Text GLabel 3150 3500 2    50   Input ~ 0
-KEY2-8
-Text GLabel 3150 3600 2    50   Input ~ 0
-KEY3-9
-Text GLabel 3150 3700 2    50   Input ~ 0
-KEY4-11
-Text GLabel 3150 3800 2    50   Input ~ 0
-KEY5-1
 $Comp
 L jamma:Jamma_Connector J1
@@
 	1    0    0    -1
 $EndComp
-Text GLabel 2650 3400 0    50   Input ~ 0
+Text GLabel 3150 3300 2    50   Input ~ 0
 COM1-2
-Text GLabel 2650 3300 0    50   Input ~ 0
+Text GLabel 3150 3200 2    50   Input ~ 0
 COM0-3
-Text GLabel 2650 3500 0    50   Input ~ 0
-COM2-6
-Text GLabel 2650 3600 0    50   Input ~ 0
-COM3-10
-Text GLabel 2650 3700 0    50   Input ~ 0
-COM4-7
 Wire Wire Line
 	2650 2900 2250 2900
@@
 Wire Wire Line
 	6650 4300 6650 4400
+Text GLabel 8050 3450 0    50   Input ~ 0
+5V
+$Comp
+L power:GND #PWR0109
+U 1 1 61C03E3B
+P 7950 3650
+F 0 "#PWR0109" H 7950 3400 50  0001 C CNN
+F 1 "GND" H 7955 3477 50  0000 C CNN
+F 2 "" H 7950 3650 50  0001 C CNN
+F 3 "" H 7950 3650 50  0001 C CNN
+	1    7950 3650
+	1    0    0    -1
+$EndComp
+Text GLabel 8050 2000 0    50   Input ~ 0
+COIN
+Text GLabel 8050 2850 0    50   Input ~ 0
+KEY5-1
+Text GLabel 8050 2750 0    50   Input ~ 0
+KEY4-11
+Text GLabel 8050 2650 0    50   Input ~ 0
+KEY3-9
+Text GLabel 8050 2550 0    50   Input ~ 0
+KEY2-8
+Text GLabel 8050 2450 0    50   Input ~ 0
+KEY1-5
+Text GLabel 8050 2350 0    50   Input ~ 0
+KEY0-4
+Text GLabel 8050 1500 0    50   Input ~ 0
+COM0-3
+Text GLabel 8050 1600 0    50   Input ~ 0
+COM1-2
+Text GLabel 8050 1700 0    50   Input ~ 0
+COM2-6
+Text GLabel 8050 1800 0    50   Input ~ 0
+COM3-10
+Text GLabel 8050 1900 0    50   Input ~ 0
+COM4-7
+$Comp
+L Connector_Generic:Conn_01x06 J3
+U 1 1 61D48DCD
+P 8250 1700
+F 0 "J3" H 8330 1692 50  0000 L CNN
+F 1 "Conn_01x06" H 8330 1601 50  0000 L CNN
+F 2 "Connector_JST:JST_EH_B6B-EH-A_1x06_P2.50mm_Vertical" H 8250 1700 50  0001 C CNN
+F 3 "~" H 8250 1700 50  0001 C CNN
+	1    8250 1700
+	1    0    0    -1
+$EndComp
+$Comp
+L Connector_Generic:Conn_01x06 J4
+U 1 1 61D4AD14
+P 8250 2550
+F 0 "J4" H 8330 2542 50  0000 L CNN
+F 1 "Conn_01x06" H 8330 2451 50  0000 L CNN
+F 2 "Connector_JST:JST_EH_B6B-EH-A_1x06_P2.50mm_Vertical" H 8250 2550 50  0001 C CNN
+F 3 "~" H 8250 2550 50  0001 C CNN
+	1    8250 2550
+	1    0    0    -1
+$EndComp
+$Comp
+L Connector_Generic:Conn_01x02 J5
+U 1 1 61D4B4F4
+P 8250 3450
+F 0 "J5" H 8330 3442 50  0000 L CNN
+F 1 "Conn_01x02" H 8330 3351 50  0000 L CNN
+F 2 "Connector_JST:JST_EH_B2B-EH-A_1x02_P2.50mm_Vertical" H 8250 3450 50  0001 C CNN
+F 3 "~" H 8250 3450 50  0001 C CNN
+	1    8250 3450
+	1    0    0    -1
+$EndComp
+Wire Wire Line
+	7950 3650 7950 3550
+Wire Wire Line
+	7950 3550 8050 3550
+Text GLabel 3150 3600 2    50   Input ~ 0
+COM4-7
+Text GLabel 3150 3500 2    50   Input ~ 0
+COM3-10
+Text GLabel 3150 3400 2    50   Input ~ 0
+COM2-6
+Text GLabel 2650 3700 0    50   Input ~ 0
+KEY5-1
+Text GLabel 2650 3600 0    50   Input ~ 0
+KEY4-11
+Text GLabel 2650 3500 0    50   Input ~ 0
+KEY3-9
+Text GLabel 2650 3400 0    50   Input ~ 0
+KEY2-8
+Text GLabel 2650 3300 0    50   Input ~ 0
+KEY1-5
+Text GLabel 2650 3200 0    50   Input ~ 0
+KEY0-4
 $EndSCHEMATC
