File: jamma_mahjong/jamma_mahjong.kicad_pcb (KiCad board)
At the start: 4 copper layers, 110.2 x 38.1 mm, 3 parts, among them J1 Jamma_Connector, J2 Mahjong_Connector, J3 Conn_02x07_Odd_Even

Commit message: x
Parts:
- added JMP1: SolderJumper_2_Open, Resistor_SMD:R_0805_2012Metric_Pad1.20x1.40mm_HandSolder, F.Cu at (213.0, 62.5)
- added SW1: SW_SPDT, SPDT:A101SYCQ04, F.Cu at (205.4, 73.8)
Connections:
- J1 pad 14: Net-(J1-Pad14) -> GND
- J1 pad E: -5V -> Net-(J1-PadE)
- J1 pad L: SPK- -> JAMMA_SPK-
- J2 pad 10: SPK- -> JONG_SPK-
- J2 pad 24: Net-(J2-Pad24) -> -5V_M
Routing:
- net -5V_M: track 0.00 -> 98.8 mm, vias 0 -> 4
- net SPK-: track 31.7 -> 0.00 mm, vias 2 -> 0
- net JAMMA_SPK-: track 0.00 -> 29.5 mm
- net JONG_SPK-: track 0.00 -> 19.5 mm, vias 0 -> 2
- net GND: track 234.0 -> 249.3 mm, vias 17 -> 15
- net 12V: track 137.6 -> 127.7 mm
- net -5V: track 0.00 -> 9.84 mm
- net TEST: track 79.9 -> 83.9 mm
- net SERVICE: track 79.2 -> 81.1 mm
- net COM4-7: track 112.9 -> 113.7 mm
Other:
- board text added: "-5V"
- board text added: "AUDIO"
- board text added: "COM 0"
- board text added: "COM 1"
- board text added: "COM 2"
- board text added: "COM 3"
- board text added: "COM 4"
- board text added: "KEY 0"
- board text added: "KEY 1"
- board text added: "KEY 2"
- board text added: "KEY 3"
- board text added: "KEY 4"
- board text added: "KEY 5"
- board text added: "Mahjong Adapter buffi - 2022"
- board text added: "SPK-"
- board text removed: "COM 0-3"
- board text removed: "COM 1-2"
- board text removed: "COM 2-6"
- board text removed: "COM 3-10"
- board text removed: "COM 4-7"
- board text removed: "KEY0-4"
- board text removed: "KEY1-5"
- board text removed: "KEY2-8"
- board text removed: "KEY3-9"
- board text removed: "KEY4-11"
- board text removed: "KEY5-1"
- board text removed: "Mahjong to Jamma adapter buffi - 2022"

Commit message: x
Parts:
- added JMP2: SolderJumper_2_Open, Resistor_SMD:R_0805_2012Metric_Pad1.20x1.40mm_HandSolder, B.Cu at (202.8, 71.8)
- added JMP3: SolderJumper_2_Open, Resistor_SMD:R_0805_2012Metric_Pad1.20x1.40mm_HandSolder, B.Cu at (202.8, 66.7)
- JMP1: moved to B.Cu
Connections:
- J1 pad 5: -5V -> Net-(J1-Pad5)
- J1 pad E: Net-(J1-PadE) -> -5V
- J2 pad 24: -5V_M -> Net-(J2-Pad24)
- J2 pad b: Net-(J2-Padb) -> -5V_M
Routing:
- net JAMMA_SPK-: track 29.5 -> 35.9 mm
- net GND: track 249.3 -> 252.4 mm
- net JONG_SPK-: track 19.5 -> 22.5 mm
Other:
- board text added: "GND SPK-"
- board text added: "JONG SPK-"

Commit message: v2
Parts:
- removed JMP2, JMP3: SolderJumper_2_Open, Resistor_SMD:R_0805_2012Metric_Pad1.20x1.40mm_HandSolder
- added J4: Conn_01x06, Connector_JST:JST_EH_B6B-EH-A_1x06_P2.50mm_Vertical, F.Cu at (176.8, 73.0)
- added J5: Conn_01x02, Connector_JST:JST_EH_B2B-EH-A_1x02_P2.50mm_Vertical, F.Cu at (227.4, 62.1)
- J3: value Conn_02x07_Odd_Even -> Conn_01x06; footprint Connector_JST:JST_PHD_B14B-PHDSS_2x07_P2.00mm_Vertical -> Connector_JST:JST_EH_B6B-EH-A_1x06_P2.50mm_Vertical
- moved SW1 14.7 mm to (194.4, 64.0), turned to -90 degrees
- moved J3 12.1 mm to (227.0, 73.0), turned to 180 degrees
- moved JMP1 3.50 mm to (213.1, 59.0)
Connections:
- J1 pad 11: Net-(J1-Pad11) -> unconnected-(J1-Pad11)
- J1 pad 17: Net-(J1-Pad17) -> KEY0-4
- J1 pad 18: COM0-3 -> KEY1-5
- J1 pad 19: COM1-2 -> KEY2-8
- J1 pad 20: COM2-6 -> KEY3-9
- J1 pad 21: COM3-10 -> KEY4-11
- J1 pad 22: COM4-7 -> KEY5-1
- J1 pad 23: Net-(J1-Pad23) -> unconnected-(J1-Pad23)
- J1 pad 24: Net-(J1-Pad24) -> unconnected-(J1-Pad24)
- J1 pad 25: Net-(J1-Pad25) -> unconnected-(J1-Pad25)
- J1 pad 26: Net-(J1-Pad26) -> unconnected-(J1-Pad26)
- J1 pad 5: Net-(J1-Pad5) -> -5V
- J1 pad 8: Net-(J1-Pad8) -> unconnected-(J1-Pad8)
- J1 pad 9: Net-(J1-Pad9) -> unconnected-(J1-Pad9)
- J1 pad J: Net-(J1-PadJ) -> unconnected-(J1-PadJ)
- J1 pad K: Net-(J1-PadK) -> unconnected-(J1-PadK)
- J1 pad M: Net-(J1-PadM) -> unconnected-(J1-PadM)
- J1 pad S: Net-(J1-PadS) -> unconnected-(J1-PadS)
- J1 pad T: Net-(J1-PadT) -> unconnected-(J1-PadT)
- J1 pad U: Net-(J1-PadU) -> COM0-3
- J1 pad V: KEY0-4 -> COM1-2
- J1 pad W: KEY1-5 -> COM2-6
- J1 pad X: KEY2-8 -> COM3-10
- J1 pad Y: KEY3-9 -> COM4-7
- J1 pad Z: KEY4-11 -> unconnected-(J1-PadZ)
- J1 pad a: KEY5-1 -> unconnected-(J1-Pada)
- J1 pad b: Net-(J1-Padb) -> unconnected-(J1-Padb)
- J1 pad c: Net-(J1-Padc) -> unconnected-(J1-Padc)
- J1 pad d: Net-(J1-Padd) -> unconnected-(J1-Padd)
- J2 pad 11: Net-(J2-Pad11) -> unconnected-(J2-Pad11)
- J2 pad 12: Net-(J2-Pad12) -> unconnected-(J2-Pad12)
- J2 pad 13: Net-(J2-Pad13) -> unconnected-(J2-Pad13)
- J2 pad 14: Net-(J2-Pad14) -> unconnected-(J2-Pad14)
- J2 pad 15: Net-(J2-Pad15) -> unconnected-(J2-Pad15)
- J2 pad 16: Net-(J2-Pad16) -> unconnected-(J2-Pad16)
- J2 pad 18: Net-(J2-Pad18) -> unconnected-(J2-Pad18)
- J2 pad 24: Net-(J2-Pad24) -> unconnected-(J2-Pad24)
- J2 pad 3: Net-(J2-Pad3) -> unconnected-(J2-Pad3)
- J2 pad 4: Net-(J2-Pad4) -> unconnected-(J2-Pad4)
- J2 pad 6: Net-(J2-Pad6) -> unconnected-(J2-Pad6)
- J2 pad D: Net-(J2-PadD) -> unconnected-(J2-PadD)
- J2 pad H: Net-(J2-PadH) -> unconnected-(J2-PadH)
- J2 pad U: Net-(J2-PadU) -> unconnected-(J2-PadU)
- J2 pad V: Net-(J2-PadV) -> unconnected-(J2-PadV)
- J3 pad 1: 5V -> COM0-3
- J3 pad 2: GND -> COM1-2
- J3 pad 3: COIN -> COM2-6
- J3 pad 4: KEY0-4 -> COM3-10
- J3 pad 5: COM0-3 -> COM4-7
- J3 pad 6: KEY1-5 -> unconnected-(J3-Pad6)
Routing:
- net GND: track 252.4 -> 150.3 mm, vias 15 -> 24
- net KEY5-1: track 115.6 -> 44.9 mm, vias 1 -> 0
- net KEY4-11: track 110.5 -> 43.4 mm, vias 1 -> 0
- net KEY3-9: track 105.3 -> 43.4 mm, vias 1 -> 0
- net KEY2-8: track 101.5 -> 43.9 mm, vias 1 -> 0
- net COIN: track 95.1 -> 42.3 mm, vias 2 -> 0
- net KEY1-5: track 103.0 -> 50.6 mm, vias 1 -> 0
- net KEY0-4: track 105.6 -> 57.2 mm, vias 1 -> 0
- net 12V: track 127.7 -> 98.1 mm, vias 5 -> 10
- net JAMMA_SPK-: track 35.9 -> 13.8 mm
- net SERVICE: track 81.1 -> 60.8 mm
- net TEST: track 83.9 -> 66.6 mm
- net COM4-7: track 113.7 -> 97.5 mm
- net COM2-6: track 109.4 -> 94.8 mm
- net COM1-2: track 112.2 -> 97.6 mm
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- added copper zone on B.Cu, net -5V
- added copper zone on F.Cu, net -5V
- added copper zone on B.Cu, net -5V_M
- added copper zone on F.Cu, net -5V_M
- added copper zone on In1.Cu, net -5V_M
- added copper zone on B.Cu, net 12V
- added copper zone on F.Cu, net 12V
- added copper zone on In1.Cu, net 12V
- added copper zone on B.Cu, net 5V
- added copper zone on F.Cu, net 5V
- added copper zone on B.Cu, net BLUE
- added copper zone on F.Cu, net BLUE
- added copper zone on In1.Cu, net BLUE
- added copper zone on B.Cu, net GND
- added copper zone on F.Cu, net GND
- added copper zone on B.Cu, net GREEN
- added copper zone on F.Cu, net GREEN
- added copper zone on In1.Cu, net GREEN
- added copper zone on B.Cu, net RED
- added copper zone on F.Cu, net RED
- added copper zone on In1.Cu, net RED
- added copper zone on B.Cu, net SYNC
- added copper zone on F.Cu, net SYNC
- added copper zone on In1.Cu, net SYNC
Other:
- board size 110.2 x 38.1 mm -> 111 x 38.8 mm
- net class Default removed
- board text added: "0"
- board text added: "1"
- board text added: "2"
- board text added: "3"
- board text added: "4"
- board text added: "5"
- board text added: "COM"
- board text added: "COM0 = P2 ST COM2 = P2 D COM4 = P2 R"
- board text added: "COM1 = P2 U COM3 = P2 L"
- board text added: "KEY"
- board text added: "KEY0 = P1 ST KEY2 = P1 D KEY4 = P1 R"
- board text added: "KEY1 = P1 U KEY3 = P1 L KEY5 = P1 B1"
- board text removed: "COIN"
- board text removed: "COM 0"
- board text removed: "COM 1"
- board text removed: "COM 2"
- board text removed: "COM 3"
- board text removed: "COM 4"
- board text removed: "COM0 = P1 U COM2 = P1 L COM4 = P1 B1"
- board text removed: "COM1 = P1 D COM3 = P1 R"
- board text removed: "GND SPK-"
- board text removed: "JONG SPK-"
- board text removed: "KEY 0"
- board text removed: "KEY 1"
- board text removed: "KEY 2"
- board text removed: "KEY 3"
- board text removed: "KEY 4"
- board text removed: "KEY 5"
- board text removed: "KEY0 = P2 U KEY2 = P2 L KEY4 = P2 B1"
- board text removed: "KEY1 = P2 D KEY3 = P2 R KEY5 = P2 B2"

Commit message: More stuff
Routing:
- net COIN: track 42.3 -> 43.0 mm
Changed lines of the file:
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@@
       (usegerberextensions true)
       (usegerberattributes false)
-      (usegerberadvancedattributes true)
-      (creategerberjobfile true)
+      (usegerberadvancedattributes false)
+      (creategerberjobfile false)
       (svguseinch false)
       (svgprecision 6)
@@
     (fp_line (start -2.5 2.2) (end 15 2.2) (layer "F.Fab") (width 0.1))
     (fp_line (start 15 -1.6) (end -2.5 -1.6) (layer "F.Fab") (width 0.1))
-    (pad "1" thru_hole roundrect locked (at 0 0 180) (size 1.7 1.95) (drill 0.95) (layers *.Cu *.Mask) (roundrect_rratio 0.147059)
+    (pad "1" thru_hole roundrect locked (at 0 0 180) (size 1.7 1.95) (drill 0.95) (layers *.Cu *.Mask) (roundrect_rratio 0.1470588235)
       (net 46 "COM0-3") (pinfunction "Pin_1") (pintype "passive"))
     (pad "2" thru_hole oval locked (at 2.5 0 180) (size 1.7 1.95) (drill 0.95) (layers *.Cu *.Mask)
@@
     (fp_line (start -2.5 2.2) (end 15 2.2) (layer "F.Fab") (width 0.1))
     (fp_line (start -2.5 -1.6) (end -2.5 2.2) (layer "F.Fab") (width 0.1))
-    (pad "1" thru_hole roundrect locked (at 0 0 180) (size 1.7 1.95) (drill 0.95) (layers *.Cu *.Mask) (roundrect_rratio 0.147059)
+    (pad "1" thru_hole roundrect locked (at 0 0 180) (size 1.7 1.95) (drill 0.95) (layers *.Cu *.Mask) (roundrect_rratio 0.1470588235)
       (net 39 "KEY0-4") (pinfunction "Pin_1") (pintype "passive"))
     (pad "2" thru_hole oval locked (at 2.5 0 180) (size 1.7 1.95) (drill 0.95) (layers *.Cu *.Mask)
@@
     (fp_line (start -2.5 -1.6) (end -2.5 2.2) (layer "F.Fab") (width 0.1))
     (fp_line (start 5 2.2) (end 5 -1.6) (layer "F.Fab") (width 0.1))
-    (pad "1" thru_hole roundrect locked (at 0 0 180) (size 1.7 2) (drill 1) (layers *.Cu *.Mask) (roundrect_rratio 0.147059)
+    (pad "1" thru_hole roundrect locked (at 0 0 180) (size 1.7 2) (drill 1) (layers *.Cu *.Mask) (roundrect_rratio 0.1470588235)
       (net 3 "5V") (pinfunction "Pin_1") (pintype "passive"))
     (pad "2" thru_hole oval locked (at 2.5 0 180) (size 1.7 2) (drill 1) (layers *.Cu *.Mask)
@@
     (fp_line (start 1 0.625) (end 1 -0.625) (layer "B.Fab") (width 0.1))
     (fp_line (start 1 -0.625) (end -1 -0.625) (layer "B.Fab") (width 0.1))
-    (pad "1" smd roundrect locked (at -1 0 90) (size 1.2 1.4) (layers "B.Cu" "B.Paste" "B.Mask") (roundrect_rratio 0.208333)
+    (pad "1" smd roundrect locked (at -1 0 90) (size 1.2 1.4) (layers "B.Cu" "B.Paste" "B.Mask") (roundrect_rratio 0.2083333333)
       (net 52 "-5V_M") (pinfunction "A") (pintype "passive"))
-    (pad "2" smd roundrect locked (at 1 0 90) (size 1.2 1.4) (layers "B.Cu" "B.Paste" "B.Mask") (roundrect_rratio 0.208333)
+    (pad "2" smd roundrect locked (at 1 0 90) (size 1.2 1.4) (layers "B.Cu" "B.Paste" "B.Mask") (roundrect_rratio 0.2083333333)
       (net 4 "-5V") (pinfunction "B") (pintype "passive"))
     (model "${KISYS3DMOD}/Resistor_SMD.3dshapes/R_0805_2012Metric.wrl"
@@
   (segment (start 202 71.9) (end 202 81.23) (width 1.5) (layer "B.Cu") (net 8))
   (segment (start 199.9 69.8) (end 202 71.9) (width 1.5) (layer "B.Cu") (net 8))
-  (segment (start 176.57548 71.57548) (end 177.63975 71.57548) (width 0.5) (layer "F.Cu") (net 9))
+  (segment (start 166.36 79.276242) (end 166.36 81.23) (width 0.5) (layer "F.Cu") (net 9))
+  (segment (start 177.65 71) (end 178.62 71.97) (width 0.5) (layer "F.Cu") (net 9))
+  (segment (start 174 69) (end 176 71) (width 0.5) (layer "F.Cu") (net 9))
+  (segment (start 176 71) (end 177.65 71) (width 0.5) (layer "F.Cu") (net 9))
+  (segment (start 178.62 74.35) (end 178.01 74.96) (width 0.5) (layer "F.Cu") (net 9))
+  (segment (start 178.01 74.96) (end 170.676242 74.96) (width 0.5) (layer "F.Cu") (net 9))
+  (segment (start 170.676242 74.96) (end 166.36 79.276242) (width 0.5) (layer "F.Cu") (net 9))
+  (segment (start 170.32 52.02) (end 170.32 55.82) (width 0.5) (layer "F.Cu") (net 9))
   (segment (start 170.32 55.82) (end 174 59.5) (width 0.5) (layer "F.Cu") (net 9))
-  (segment (start 170.32 52.02) (end 170.32 55.82) (width 0.5) (layer "F.Cu") (net 9))
-  (segment (start 171.211722 74.42452) (end 166.36 79.276242) (width 0.5) (layer "F.Cu") (net 9))
-  (segment (start 166.36 79.276242) (end 166.36 81.23) (width 0.5) (layer "F.Cu") (net 9))
-  (segment (start 178.04952 71.98525) (end 178.04952 74.01475) (width 0.5) (layer "F.Cu") (net 9))
-  (segment (start 177.63975 74.42452) (end 175.86025 74.42452) (width 0.5) (layer "F.Cu") (net 9))
-  (segment (start 177.63975 71.57548) (end 178.04952 71.98525) (width 0.5) (layer "F.Cu") (net 9))
-  (segment (start 175.45048 74.01475) (end 175.45048 73.762318) (width 0.5) (layer "F.Cu") (net 9))
-  (segment (start 175.45048 73.762318) (end 174.788278 74.42452) (width 0.5) (layer "F.Cu") (net 9))
-  (segment (start 174.788278 74.42452) (end 171.211722 74.42452) (width 0.5) (layer "F.Cu") (net 9))
-  (segment (start 175.86025 74.42452) (end 175.45048 74.01475) (width 0.5) (layer "F.Cu") (net 9))
-  (segment (start 174 69) (end 176.57548 71.57548) (width 0.5) (layer "F.Cu") (net 9))
+  (segment (start 178.62 71.97) (end 178.62 74.35) (width 0.5) (layer "F.Cu") (net 9))
   (segment (start 174 59.5) (end 174 69) (width 0.5) (layer "F.Cu") (net 9))
-  (segment (start 178.04952 74.01475) (end 177.63975 74.42452) (width 0.5) (layer "F.Cu") (net 9))
   (segment (start 202 69.412) (end 202 81.23) (width 1.5) (layer "F.Cu") (net 10))
   (segment (start 199.898 67.31) (end 202 69.412) (width 1.5) (layer "F.Cu") (net 10))
